File: kicad/SpeakerProtect_LeeKnatta.kicad_pcb (KiCad board)
At the start: 2 copper layers, 102 parts, among them J1 Conn_01x02_Pin, J2 Conn_01x02_Pin, J3 Conn_01x02_Pin, J4 Conn_01x02_Pin, J5 Conn_01x02_Pin, J6 Conn_01x02_Pin, J7 Conn_01x02_Pin, Q1 2N5401, Q2 2N5401, Q22 BC557, Q23 MJE350, Q25 2N5551, Q40 2N5551, Q41 2N5401, Q42 BC557, Q43 BC547, Q44 MJE350, Q45 MJE340, Q46 2N5551, Q47 2N5401, Q48 BC557, Q49 BC547, Q50 MJE350, Q51 MJE340, Q60 BC547, Q61 MJE340, Q62 IXFK150N30X3, Q63 IXFK150N30X3, Q64 IXFK150N30X3, Q65 IXFK150N30X3, Q70 2N5551, Q71 BC557, Q73 MJE350, Q80 2N5551, Q81 2N5551, Q82 2N5551, T1 Transformer_1P_1S, U1 AQY280EH, U2 AQY280EH, U3 AQY280EH, U4 AQY280EH, U60 ASSR-V621-002E, U61 ASSR-V621-002E

Commit message: Completed PCB
Parts:
- added J10: ~, ACRM:Spade_Connector, F.Cu at (202.2, 76.2)
- added J11: ~, ACRM:Spade_Connector, F.Cu at (202.2, 59.4)
- added J12: ~, ACRM:Spade_Connector, F.Cu at (202.2, 45.0)
- added J8: ~, ACRM:Spade_Connector, F.Cu at (224.1, 45.0)
- added J9: ~, ACRM:Spade_Connector, F.Cu at (202.2, 90.7)
- added REF**: MountingHole_3.2mm_M3, MountingHole:MountingHole_3.2mm_M3, F.Cu at (226.2, 40.3)
- added REF**: MountingHole_3.2mm_M3, MountingHole:MountingHole_3.2mm_M3, F.Cu at (52.3, 96.6)
- added REF**: MountingHole_3.2mm_M3, MountingHole:MountingHole_3.2mm_M3, F.Cu at (52.3, 40.0)
- added REF**: MountingHole_3.2mm_M3, MountingHole:MountingHole_3.2mm_M3, F.Cu at (226.2, 96.9)
- C1: renamed from C83; footprint Capacitor_THT:CP_Radial_D5.0mm_P2.50mm -> Capacitor_THT:CP_Radial_D10.0mm_P5.00mm_P7.50mm
- C40, C43: footprint Capacitor_THT:CP_Radial_D5.0mm_P2.50mm -> Capacitor_THT:CP_Radial_D5.0mm_P2.00mm
- C41, C42, C44, C45, C82: footprint Capacitor_THT:C_Rect_L7.0mm_W2.0mm_P5.00mm -> Capacitor_THT:C_Rect_L7.0mm_W4.5mm_P5.00mm
- C80: footprint Capacitor_THT:CP_Radial_D5.0mm_P2.50mm -> Capacitor_THT:C_Rect_L7.2mm_W5.0mm_P5.00mm
- C81: footprint Capacitor_THT:CP_Radial_D5.0mm_P2.50mm -> Capacitor_THT:CP_Radial_D16.0mm_P7.50mm
- D80: footprint Diode_THT:Diode_Bridge_32.0x5.6x17.0mm_P10.0mm_P7.5mm -> ACRM:Diode_Bridge_14.5x3.5x10.5mm_P3.61
- D83: footprint Diode_THT:D_DO-35_SOD27_P7.62mm_Horizontal -> Diode_THT:D_DO-41_SOD81_P2.54mm_Vertical_CathodeUp
- J1, J2, J3, J4, J5: value Conn_01x02_Pin -> ~; footprint TerminalBlock_4Ucon:TerminalBlock_4Ucon_1x02_P3.50mm_Horizontal -> ACRM:Spade_Connector
- Q1, Q2, Q22, Q25, Q40, Q41, Q42, Q43, Q46, Q47, Q48, Q49, Q60, Q70, Q71, Q80, Q81, Q82: footprint Package_TO_SOT_THT:TO-92_Inline -> Package_TO_SOT_THT:TO-92_Inline_Wide
- R46, R47, R50, R51, R72, R81: footprint Resistor_THT:R_Axial_DIN0207_L6.3mm_D2.5mm_P10.16mm_Horizontal -> Resistor_THT:R_Axial_DIN0207_L6.3mm_D2.5mm_P2.54mm_Vertical
- T1: footprint Transformer_THT:Transformer_CHK_EI48-8VA_1xSec -> ACRM:Transformer_Myrra-44233-230V-18V-5VA-37x44
- moved J2 236.2 mm to (46.9, 53.3), turned to 90 degrees
- moved R48 188.1 mm to (157.1, 39.8), turned to 180 degrees
- moved D43 183.4 mm to (147.0, 43.8)
- moved R41 182.1 mm to (144.1, 39.3), turned to -90 degrees
- moved D23 174.8 mm to (147.0, 59.7)
- moved R49 166.5 mm to (147.0, 63.7)
- moved C44 162.7 mm to (170.1, 44.0), turned to 90 degrees
- moved Q47 161.8 mm to (149.4, 55.1)
- moved Q49 161.7 mm to (157.0, 58.7)
- moved C43 161.5 mm to (144.4, 54.8)
- moved R50 160.3 mm to (160.6, 49.8), turned to 180 degrees
- moved Q46 160.0 mm to (149.4, 49.0)
- moved R51 159.2 mm to (158.5, 53.6)
- moved Q51 158.3 mm to (165.4, 63.0), turned to 180 degrees
- moved Q50 157.3 mm to (160.8, 40.5)
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Connections:
- D80 pad 2: AC_IN_2 -> AC_IN_1
- D80 pad 3: AC_IN_1 -> AC_IN_2
- J1 pad 1: Net-(J1-Pin_1) -> Net-(T1-AA)
- J1 pad 2: Net-(J1-Pin_2) -> Net-(T1-AA)
- J2 pad 1: AMP_LEFT_GND -> Net-(T1-AB)
- J2 pad 2: AMP_LEFT -> Net-(T1-AB)
- J3 pad 1: AMP_RIGHT_GND -> AMP_LEFT
- J3 pad 2: AMP_RIGHT -> AMP_LEFT
- J4 pad 1: GND -> AMP_LEFT_GND
- J4 pad 2: AMP_LEFT_OUT -> AMP_LEFT_GND
- J5 pad 1: GND -> AMP_RIGHT
- J5 pad 2: AMP_RIGHT_OUT -> AMP_RIGHT
- R1 pad 2: Net-(R1-Pad2) -> SHUTDOWN
- R2 pad 1: Net-(R1-Pad2) -> SHUTDOWN
- T1 pad 1: Net-(J1-Pin_1) -> Net-(T1-AA)
- T1 pad 2: Net-(J1-Pin_2) -> Net-(T1-AB)
Routing:
- net GND: track 0.00 -> 474.2 mm
- net +SUPPLY: track 0.00 -> 290.1 mm
- net SHUTDOWN: track 0.00 -> 139.2 mm
- net RELAY_ENABLE: track 0.00 -> 135.2 mm
- net AMP_RIGHT: track 0.00 -> 131.1 mm
- net AMP_LEFT: track 0.00 -> 129.6 mm
- net AMP_LEFT_GND: track 0.00 -> 100.0 mm
- net AMP_RIGHT_GND: track 0.00 -> 99.9 mm
- net DC_FAULT_R: track 0.00 -> 94.3 mm
- net DC_FAULT_L: track 0.00 -> 90.8 mm
- net AC_IN_2: track 0.00 -> 84.5 mm
- net DC_ENABLE_L: track 0.00 -> 77.0 mm
- net AC_IN_1: track 0.00 -> 63.9 mm
- net DC_ENABLE_R: track 0.00 -> 55.8 mm
- net Net-(U60-Pad4): track 0.00 -> 40.9 mm
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- added copper zone on B.Cu, net GND
Other:
- board outline added: 182 x 69 mm
- board text added: "- +"
- board text added: "AC Loss"
- board text added: "Amp Left"
- board text added: "Amp Left Gnd"
- board text added: "Amp Right"
- board text added: "Amp Right Gnd"
- board text added: "DC Detect Left"
- board text added: "DC Detect Right"
- board text added: "Lee Knatta Speaker Protect PCB V1.0 acramonics 10/26"
- board text added: "Mains In"
- board text added: "PSU"
- board text added: "RED LED"
- board text added: "Solid State Relay"
- board text added: "Spk Left"
- board text added: "Spk Left Gnd"
- board text added: "Spk Right"
- board text added: "Spk Right Gnd"
- board text added: "Startup Delay"
- board text added: "Status Indication"
