File: kicad/SpeakerProtect_LeeKnatta.kicad_sch (KiCad schematic)
At the start: 0 parts

Commit message: Added more schematics
Parts:
- added C40, C43: 33uF 16V NP, Package_TO_SOT_THT:TO-92_Inline, symbol Device:C_Polarized_Small
- added C41, C42, C44, C45: 1nF, Package_TO_SOT_THT:TO-92_Inline, symbol Device:C_Small
- added C80: 100nF 250V, Package_TO_SOT_THT:TO-92_Inline, symbol Device:C_Small
- added C81: 470uF 100V, Package_TO_SOT_THT:TO-92_Inline, symbol Device:C_Polarized_Small
- added C82: 330nF, Package_TO_SOT_THT:TO-92_Inline, symbol Device:C_Small
- added C83: 82uF 100V, Package_TO_SOT_THT:TO-92_Inline, symbol Device:C_Polarized_Small
- added D2: LED, LED_SMD:LED_Cree-XHP50_3V_HighDensity, symbol Device:LED
- added D20, D22, D23, D42, D43, D81, D83, D84, D85: BAV21, Diode_THT:D_DO-35_SOD27_P7.62mm_Horizontal, symbol Diode:BAV21
- added D80: KBP206G, Diode_THT:Diode_Bridge_32.0x5.6x17.0mm_P10.0mm_P7.5mm, symbol Diode_Bridge:B40C3x00-2200A
- added Q1, Q2, Q41, Q47: 2N5401, Package_TO_SOT_THT:TO-92_Inline, symbol Transistor_BJT:2N3905
- added Q22, Q42, Q48: BC557, Package_TO_SOT_THT:TO-92_Inline, symbol Transistor_BJT:BC557
- added Q23, Q44, Q50: MJE350, Package_TO_SOT_THT:TO-126-3_Vertical, symbol Transistor_BJT:BD436
- added Q25, Q40, Q46, Q80, Q81, Q82: 2N5551, Package_TO_SOT_THT:TO-92_Inline, symbol Transistor_BJT:2N3904
- added Q43, Q49: BC547, Package_TO_SOT_THT:TO-92_Inline, symbol Transistor_BJT:BC547
- added Q45, Q51: MJE340, Package_TO_SOT_THT:TO-126-3_Vertical, symbol Transistor_BJT:BD135
- added R1, R12, R26, R3, R31, R40, R41, R44, R45, R48, R49, R5, R83: 100K, symbol Device:R_Small
- added R11, R13: 20K, symbol Device:R_Small
- added R2, R27, R46, R47, R50, R51, R6, R84: 100R, symbol Device:R_Small
- added R20, R21: 0R, symbol Device:R_Small
- added R4, R7, R81: 47K5, symbol Device:R_Small
- added R4: 2K, symbol Device:R_Small
- added R80: 10K, symbol Device:R_Small
- added U1, U2, U3, U4: AQY280EH, Package_DIP:DIP-4_W7.62mm, symbol Relay_SolidState:AQY280EH
Connections:
- new net: Q49.2 (B), Q51.1 (E), R51.1
- new net: C45.2, D23.2 (A), Q49.3 (E), R51.2
- new net: Q43.2 (B), Q45.1 (E), R47.1
- new net: C42.2, D22.2 (A), Q43.3 (E), R47.2
- new net: Q50.2 (C), U3.1
- new net: C41.1, D42.1 (K), Q42.3 (E), R46.1
- new net: C41.2, Q42.1 (C), Q44.3 (B), R44.1
- new net: C82.1, D83.2 (A), R83.2, R84.1
- new net: Q80.3 (C), R84.2
- new net: Q80.2 (B), R4.1, R81.2
- new net: Q41.3 (C), R45.1
- new net: C42.1, Q43.1 (C), Q45.3 (B), R45.2
- new net: C43.1, Q46.2 (B), Q47.2 (B), R41.2
- new net: R1.2, R2.1
- new net: Q42.2 (B), Q44.1 (E), R46.2
- new net: Q44.2 (C), U2.1
- new net: D81.1 (K), D84.1 (K), R81.1
- new net: D20.1 (K), R20.1, R21.1
- new net: C44.2, Q48.1 (C), Q50.3 (B), R48.1
- new net: Q48.2 (B), Q50.1 (E), R50.2
- new net: C44.1, D43.1 (K), Q48.3 (E), R50.1
- new net: Q51.2 (C), U4.2
- new net: C45.1, Q49.1 (C), Q51.3 (B), R49.2
- new net: C40.1, Q40.2 (B), Q41.2 (B), R40.2
- new net: Q40.3 (C), R44.2
- new net: Q25.2 (B), R31.2
- new net: Q82.2 (B), R11.2
- new net: Q22.1 (C), Q23.3 (B), R26.1
- new net: D20.2 (A), R26.2
- new net: Q2.2 (B), R5.2, R6.1
- new net: Q22.2 (B), Q23.1 (E), R27.2
- new net: Q47.3 (C), R49.1
- new net: D83.1 (K), Q81.2 (B)
- new net: Q46.3 (C), R48.2
- new net: Q45.2 (C), U1.2
- new net: C83.1, R2.2
- new net: C80.1, R80.2
- new net: Q2.3 (C), R11.1, R12.1, R13.1
- new net: Q1.1 (E), Q2.1 (E), R4.2
- new net: Q1.3 (C), R6.2, R7.1
- new net: Q1.2 (B), R3.2
- new net: D2.2 (A), Q23.2 (C), R31.1
- new net +SUPPLY: C81.1, D80.4 (+), D85.1 (K), Q22.3 (E), R1.1, R27.1, R4.1, R5.1, R83.1
- new net AC_IN_1: D80.3, D84.2 (A), R80.1
- new net AC_IN_2: C80.2, D80.2, D81.2 (A)
- new net AMP_LEFT: D22.1 (K), D42.2 (A), R40.1
- new net AMP_LEFT_GND: C40.2, Q40.1 (E), Q41.1 (E), U1.1, U2.2
- new net AMP_RIGHT: D23.1 (K), D43.2 (A), R41.1
- new net AMP_RIGHT_GND: C43.2, Q46.1 (E), Q47.1 (E), U3.2, U4.1
- new net AUX_CONTROL: Q82.3 (C)
- new net DC_ENABLE_L: C81.2, C82.2, C83.2, D2.1 (K), D80.1 (-), Q25.1 (E), Q80.1 (E), Q81.1 (E), Q82.1 (E), R4.2, R7.2, U1.3, U2.3, U3.3, U4.3
- new net DC_FAULT_L: R20.2, U1.4, U2.4
- new net DC_FAULT_R: R21.2, U3.4, U4.4
- new net RELAY_ENABLE: R13.2
- new net RELAY_STATUS: R12.2
- new net SHUTDOWN: D85.2 (A), Q25.3 (C), Q81.3 (C), R3.1

Commit message: Added HiFiSonix design
Parts:
- added D60, D61: BZX55B18, Package_DIP:DIP-40_W15.24mm, symbol Device:D_Zener
- added D70: LED-Green, symbol Device:LED
- added Q60: BC547, Package_TO_SOT_THT:TO-92_Inline, symbol Transistor_BJT:BC547
- added Q61: MJE340, Package_TO_SOT_THT:TO-126-3_Vertical, symbol Transistor_BJT:BD135
- added Q62, Q63, Q64, Q65: IXFK150N30X3, Package_TO_SOT_THT:TO-247-3_Vertical, symbol ACRM:IXFK150N30X3
- added Q70: 2N5551, Package_TO_SOT_THT:TO-92_Inline, symbol Transistor_BJT:2N3904
- added Q71: BC557, Package_TO_SOT_THT:TO-92_Inline, symbol Transistor_BJT:BC557
- added Q73: MJE350, Package_TO_SOT_THT:TO-126-3_Vertical, symbol Transistor_BJT:BD436
- added R18, R19: 0R, Resistor_THT:R_Array_SIP4, symbol Device:R_Small
- added R60: 27R4, symbol Device:R_Small
- added R71: 100K, symbol Device:R_Small
- added R72: 100R, symbol Device:R_Small
- added RV63, RV64: 270V, Package_QFP:TQFP-44_10x10mm_P0.8mm, symbol Device:Varistor
- added U60, U61: ASSR-V621-002E, Package_DIP:DIP-8_W7.62mm, symbol ACRM:ASSR-V621-002E
- renumbered R4 to R82
Connections:
- net +SUPPLY: now also Q71.3 (E), R72.1, U60.1
- net AMP_LEFT: now also Q62.2 (D), RV63.1
- net AMP_RIGHT: now also Q64.2 (D), RV64.1
- net DC_ENABLE_L: now also R19.2; no longer C81.2, C82.2, C83.2, D2.1 (K), D80.1 (-), Q25.1 (E), Q80.1 (E), Q81.1 (E), Q82.1 (E), R7.2, R82.2, U3.3, U4.3
- net RELAY_ENABLE: now also Q60.1 (C), Q61.3 (B)
- net RELAY_STATUS: now also Q70.2 (B)
- new net: Q71.1 (C), Q73.3 (B), R71.1
- new net: Q71.2 (B), Q73.1 (E), R72.2
- new net: D60.1 (K), Q62.1 (G), Q63.1 (G), U60.8
- new net: D60.2 (A), Q62.3 (S), Q63.3 (S), U60.5
- new net: Q60.2 (B), Q61.1 (E), R60.1
- new net: Q61.2 (C), U61.4
- new net: U60.4, U61.1
- new net: U61.2, U61.3
- new net: D61.2 (A), Q64.3 (S), Q65.3 (S), U61.5
- new net: U61.6, U61.7
- new net: D61.1 (K), Q64.1 (G), Q65.1 (G), U61.8
- new net: D70.2 (A), Q73.2 (C)
- new net: Q70.3 (C), R71.2
- new net: U60.2, U60.3
- new net: U60.6, U60.7
- new net AMP_LEFT_OUT: Q63.2 (D), Q65.2 (D), RV63.2, RV64.2
- new net DC_ENABLE_R: R18.2, U3.3, U4.3
- new net GND: C81.2, C82.2, C83.2, D2.1 (K), D70.1 (K), D80.1 (-), Q25.1 (E), Q60.3 (E), Q70.1 (E), Q80.1 (E), Q81.1 (E), Q82.1 (E), R18.1, R19.1, R60.2, R7.2, R82.2

Commit message: Added connections and started PCB
Parts:
- added J6, J7: Conn_01x02_Pin, TerminalBlock_4Ucon:TerminalBlock_4Ucon_1x02_P3.50mm_Horizontal, symbol Connector:Conn_01x02_Pin
- C40, C43: value 33uF 16V NP -> 47uF 16V NP; footprint Package_TO_SOT_THT:TO-92_Inline -> Capacitor_THT:CP_Radial_D5.0mm_P2.50mm
- C41, C42, C44, C45, C82: footprint Package_TO_SOT_THT:TO-92_Inline -> Capacitor_THT:C_Rect_L7.0mm_W2.0mm_P5.00mm
- C80, C81, C83: footprint Package_TO_SOT_THT:TO-92_Inline -> Capacitor_THT:CP_Radial_D5.0mm_P2.50mm
- D2: value LED -> LED-Red; footprint LED_SMD:LED_Cree-XHP50_3V_HighDensity -> (none)
- D60, D61: footprint Package_DIP:DIP-40_W15.24mm -> Diode_THT:D_DO-35_SOD27_P7.62mm_Horizontal
- D70: value LED-Green -> LED-G
- R1, R11, R12, R13, R2, R20, R21, R26, R27, R3, R31, R4, R40, R41, R44, R45, R46, R47, R48, R49, R5, R50, R51, R6, R60, R7, R71, R72, R80, R81, R82, R83, R84: footprint (none) -> Resistor_THT:R_Axial_DIN0207_L6.3mm_D2.5mm_P10.16mm_Horizontal
- R18, R19: footprint Resistor_THT:R_Array_SIP4 -> Resistor_THT:R_Axial_DIN0207_L6.3mm_D2.5mm_P10.16mm_Horizontal
- RV63, RV64: footprint Package_QFP:TQFP-44_10x10mm_P0.8mm -> Varistor:RV_Disc_D15.5mm_W7.5mm_P7.5mm
Connections:
- net AMP_LEFT_OUT: no longer Q65.2 (D), RV64.2
- net GND: now also J6.1 (Pin_1), J7.1 (Pin_1)
- net at D70.2 (A), Q73.2 (C): now also J7.2 (Pin_2)
- net at D2.2 (A), Q23.2 (C), R31.1: now also J6.2 (Pin_2)
- new net AMP_RIGHT_OUT: Q65.2 (D), RV64.2
Other:
- added sheet Connections (connections.kicad_sch)
- note added: "Q61 needs a small heatsink"
- moved on the sheet: D70, Q70, Q71, Q73, R71, R72

Commit message: Completed PCB
Parts:
- C1: renamed from C83; footprint Capacitor_THT:CP_Radial_D5.0mm_P2.50mm -> Capacitor_THT:CP_Radial_D10.0mm_P5.00mm_P7.50mm
- C40, C43: footprint Capacitor_THT:CP_Radial_D5.0mm_P2.50mm -> Capacitor_THT:CP_Radial_D5.0mm_P2.00mm
- C41, C42, C44, C45, C82: footprint Capacitor_THT:C_Rect_L7.0mm_W2.0mm_P5.00mm -> Capacitor_THT:C_Rect_L7.0mm_W4.5mm_P5.00mm
- C80: footprint Capacitor_THT:CP_Radial_D5.0mm_P2.50mm -> Capacitor_THT:C_Rect_L7.2mm_W5.0mm_P5.00mm
- C81: footprint Capacitor_THT:CP_Radial_D5.0mm_P2.50mm -> Capacitor_THT:CP_Radial_D16.0mm_P7.50mm
- D80: footprint Diode_THT:Diode_Bridge_32.0x5.6x17.0mm_P10.0mm_P7.5mm -> ACRM:Diode_Bridge_14.5x3.5x10.5mm_P3.61
- D83: footprint Diode_THT:D_DO-35_SOD27_P7.62mm_Horizontal -> Diode_THT:D_DO-41_SOD81_P2.54mm_Vertical_CathodeUp
- Q1, Q2, Q22, Q25, Q40, Q41, Q42, Q43, Q46, Q47, Q48, Q49, Q60, Q70, Q71, Q80, Q81, Q82: footprint Package_TO_SOT_THT:TO-92_Inline -> Package_TO_SOT_THT:TO-92_Inline_Wide
- R46, R47, R50, R51, R72, R81: footprint Resistor_THT:R_Axial_DIN0207_L6.3mm_D2.5mm_P10.16mm_Horizontal -> Resistor_THT:R_Axial_DIN0207_L6.3mm_D2.5mm_P2.54mm_Vertical
Connections:
- net AC_IN_1: now also D80.2; no longer D80.3
- net AC_IN_2: now also D80.3; no longer D80.2
- net SHUTDOWN: now also R1.2, R2.1
Other:
- moved on the sheet: D80
Changed lines of the file:
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@@
 	)
 	(junction
+		(at 119.38 29.21)
+		(diameter 0)
+		(color 0 0 0 0)
+	)
+	(junction
 		(at 144.78 49.53)
 		(diameter 0)
@@
 	(wire
 		(pts
+			(xy 119.38 29.21) (xy 132.08 29.21)
+		)
+		(stroke
+			(width 0)
+			(type default)
+		)
+	)
+	(wire
+		(pts
 			(xy 176.53 73.66) (xy 190.5 73.66)
 		)
@@
 	(wire
 		(pts
+			(xy 119.38 29.21) (xy 119.38 30.48)
+		)
+		(stroke
+			(width 0)
+			(type default)
+		)
+	)
+	(wire
+		(pts
 			(xy 237.49 48.26) (xy 237.49 53.34)
 		)
@@
 	(wire
 		(pts
-			(xy 114.3 29.21) (xy 132.08 29.21)
+			(xy 114.3 29.21) (xy 119.38 29.21)
 		)
 		(stroke
@@
 	(wire
 		(pts
-			(xy 119.38 26.67) (xy 119.38 30.48)
+			(xy 119.38 26.67) (xy 119.38 29.21)
 		)
 		(stroke
@@
 			)
 		)
-		(property "Footprint" "Resistor_THT:R_Axial_DIN0207_L6.3mm_D2.5mm_P10.16mm_Horizontal"
+		(property "Footprint" "Resistor_THT:R_Axial_DIN0207_L6.3mm_D2.5mm_P2.54mm_Vertical"
 			(at 161.29 154.94 0)
 			(hide yes)
@@
 			)
 		)
-		(property "Footprint" "Resistor_THT:R_Axial_DIN0207_L6.3mm_D2.5mm_P10.16mm_Horizontal"
+		(property "Footprint" "Resistor_THT:R_Axial_DIN0207_L6.3mm_D2.5mm_P2.54mm_Vertical"
 			(at 72.39 154.94 0)
 			(hide yes)
@@
 			)
 		)
-		(property "Footprint" "Capacitor_THT:C_Rect_L7.0mm_W2.0mm_P5.00mm"
+		(property "Footprint" "Capacitor_THT:C_Rect_L7.0mm_W4.5mm_P5.00mm"
 			(at 52.07 91.44 0)
 			(hide yes)
@@
 			)
 		)
-		(property "Footprint" "Package_TO_SOT_THT:TO-92_Inline"
+		(property "Footprint" "Package_TO_SOT_THT:TO-92_Inline_Wide"
 			(at 99.06 155.575 0)
 			(hide yes)
@@
 			)
 		)
-		(property "Footprint" "Package_TO_SOT_THT:TO-92_Inline"
+		(property "Footprint" "Package_TO_SOT_THT:TO-92_Inline_Wide"
 			(at 52.07 64.135 0)
 			(hide yes)
@@
 			)
 		)
-		(property "Footprint" "Capacitor_THT:CP_Radial_D5.0mm_P2.50mm"
+		(property "Footprint" "Capacitor_THT:CP_Radial_D5.0mm_P2.00mm"
 			(at 124.46 118.11 0)
 			(hide yes)
@@
 			)
 		)
-		(property "Footprint" "Capacitor_THT:CP_Radial_D5.0mm_P2.50mm"
+		(property "Footprint" "Capacitor_THT:CP_Radial_D16.0mm_P7.50mm"
 			(at 64.77 29.21 0)
 			(hide yes)
@@
 			)
 		)
-		(property "Footprint" "Package_TO_SOT_THT:TO-92_Inline"
+		(property "Footprint" "Package_TO_SOT_THT:TO-92_Inline_Wide"
 			(at 59.69 93.345 0)
 			(hide yes)
@@
 			)
 		)
-		(property "Footprint" "Package_TO_SOT_THT:TO-92_Inline"
+		(property "Footprint" "Package_TO_SOT_THT:TO-92_Inline_Wide"
 			(at 148.59 93.345 0)
 			(hide yes)
@@
 			)
 		)
-		(property "Footprint" "Resistor_THT:R_Axial_DIN0207_L6.3mm_D2.5mm_P10.16mm_Horizontal"
+		(property "Footprint" "Resistor_THT:R_Axial_DIN0207_L6.3mm_D2.5mm_P2.54mm_Vertical"
 			(at 36.83 54.61 0)
 			(hide yes)
@@
 			)
 		)
-		(property "Footprint" "Capacitor_THT:C_Rect_L7.0mm_W2.0mm_P5.00mm"
+		(property "Footprint" "Capacitor_THT:C_Rect_L7.0mm_W4.5mm_P5.00mm"
 			(at 52.07 153.67 0)
 			(hide yes)
@@
 			)
 		)
-		(property "Footprint" "Resistor_THT:R_Axial_DIN0207_L6.3mm_D2.5mm_P10.16mm_Horizontal"
+		(property "Footprint" "Resistor_THT:R_Axial_DIN0207_L6.3mm_D2.5mm_P2.54mm_Vertical"
 			(at 72.39 91.44 0)
 			(hide yes)
@@
 			)
 		)
-		(property "Footprint" "Package_TO_SOT_THT:TO-92_Inline"
+		(property "Footprint" "Package_TO_SOT_THT:TO-92_Inline_Wide"
 			(at 54.61 116.205 0)
 			(hide yes)
@@
 			)
 		)
-		(property "Footprint" "Package_TO_SOT_THT:TO-92_Inline"
+		(property "Footprint" "Package_TO_SOT_THT:TO-92_Inline_Wide"
 			(at 267.97 55.245 0)
 			(hide yes)
@@
 			)
 		)
-		(property "Footprint" "Package_TO_SOT_THT:TO-92_Inline"
+		(property "Footprint" "Package_TO_SOT_THT:TO-92_Inline_Wide"
 			(at 179.07 67.945 0)
 			(hide yes)
@@
 			)
 		)
-		(property "Footprint" "Package_TO_SOT_THT:TO-92_Inline"
+		(property "Footprint" "Package_TO_SOT_THT:TO-92_Inline_Wide"
 			(at 104.14 179.705 0)
 			(hide yes)
@@
 	(symbol
 		(lib_id "Diode_Bridge:B40C3x00-2200A")
-		(at 48.26 27.94 180)
+		(at 48.26 27.94 0)
+		(mirror y)
 		(unit 1)
 		(body_style 1)
@@
 		(in_pos_files yes)
 		(dnp no)
-		(fields_autoplaced yes)
 		(property "Reference" "D80"
-			(at 59.69 21.5198 0)
+			(at 59.69 34.3602 0)
 			(show_name no)
 			(do_not_autoplace no)
@@
 		)
 		(property "Value" "KBP206G"
-			(at 59.69 24.0598 0)
+			(at 59.69 31.8202 0)
 			(show_name no)
 			(do_not_autoplace no)
@@
 			)
 		)
-		(property "Footprint" "Diode_THT:Diode_Bridge_32.0x5.6x17.0mm_P10.0mm_P7.5mm"
-			(at 44.45 31.115 0)
+		(property "Footprint" "ACRM:Diode_Bridge_14.5x3.5x10.5mm_P3.61"
+			(at 44.45 24.765 0)
 			(hide yes)
 			(show_name no)
@@
 			)
 		)
-		(property "Datasheet" "https://diotec.com/tl_files/diotec/files/pdf/datasheets/b40c3700"
+		(property "Datasheet" ""
 			(at 48.26 27.94 0)
 			(hide yes)
@@
 			)
 		)
-		(property "Footprint" "Package_TO_SOT_THT:TO-92_Inline"
+		(property "Footprint" "Package_TO_SOT_THT:TO-92_Inline_Wide"
 			(at 240.03 26.035 0)
 			(hide yes)
@@
 			)
 		)
-		(property "Footprint" "Resistor_THT:R_Axial_DIN0207_L6.3mm_D2.5mm_P10.16mm_Horizontal"
+		(property "Footprint" "Resistor_THT:R_Axial_DIN0207_L6.3mm_D2.5mm_P2.54mm_Vertical"
 			(at 111.76 153.67 0)
 			(hide yes)
@@
 			)
 		)
-		(property "Footprint" "Package_TO_SOT_THT:TO-92_Inline"
+		(property "Footprint" "Package_TO_SOT_THT:TO-92_Inline_Wide"
 			(at 59.69 153.035 0)
 			(hide yes)
@@
 			)
 		)
-		(property "Footprint" "Package_TO_SOT_THT:TO-92_Inline"
+		(property "Footprint" "Package_TO_SOT_THT:TO-92_Inline_Wide"
 			(at 143.51 130.175 0)
 			(hide yes)
@@
 			)
 		)
-		(property "Footprint" "Diode_THT:D_DO-35_SOD27_P7.62mm_Horizontal"
+		(property "Footprint" "Diode_THT:D_DO-41_SOD81_P2.54mm_Vertical_CathodeUp"
 			(at 75.565 54.61 0)
 			(hide yes)
@@
 			)
 		)
-		(property "Footprint" "Package_TO_SOT_THT:TO-92_Inline"
+		(property "Footprint" "Package_TO_SOT_THT:TO-92_Inline_Wide"
 			(at 143.51 116.205 0)
 			(hide yes)
@@
 			)
 		)
-		(property "Footprint" "Resistor_THT:R_Axial_DIN0207_L6.3mm_D2.5mm_P10.16mm_Horizontal"
+		(property "Footprint" "Resistor_THT:R_Axial_DIN0207_L6.3mm_D2.5mm_P2.54mm_Vertical"
 			(at 161.29 91.44 0)
 			(hide yes)
@@
 			)
 		)
-		(property "Footprint" "Package_TO_SOT_THT:TO-92_Inline"
+		(property "Footprint" "Package_TO_SOT_THT:TO-92_Inline_Wide"
 			(at 148.59 153.035 0)
 			(hide yes)
@@
 			)
 		)
-		(property "Footprint" "Capacitor_THT:C_Rect_L7.0mm_W2.0mm_P5.00mm"
+		(property "Footprint" "Capacitor_THT:C_Rect_L7.0mm_W4.5mm_P5.00mm"
 			(at 140.97 91.44 0)
 			(hide yes)
@@
 			)
 		)
-		(property "Footprint" "Capacitor_THT:CP_Radial_D5.0mm_P2.50mm"
+		(property "Footprint" "Capacitor_THT:C_Rect_L7.2mm_W5.0mm_P5.00mm"
 			(at 25.4 31.75 0)
 			(hide yes)
@@
 			)
 		)
-		(property "Footprint" "Capacitor_THT:C_Rect_L7.0mm_W2.0mm_P5.00mm"
+		(property "Footprint" "Capacitor_THT:C_Rect_L7.0mm_W4.5mm_P5.00mm"
 			(at 64.77 73.66 0)
 			(hide yes)
@@
 		(dnp no)
 		(fields_autoplaced yes)
-		(property "Reference" "C83"
+		(property "Reference" "C1"
 			(at 121.92 54.0638 0)
 			(show_name no)
@@
 			)
 		)
-		(property "Footprint" "Capacitor_THT:CP_Radial_D5.0mm_P2.50mm"
+		(property "Footprint" "Capacitor_THT:CP_Radial_D10.0mm_P5.00mm_P7.50mm"
 			(at 119.38 55.88 0)
 			(hide yes)
@@
 			(project "SpeakerProtect_LeeKnatta"
 				(path "/1c068ca8-5f29-49e1-8ff3-7a0995a53dab"
-					(reference "C83")
+					(reference "C1")
 					(unit 1)
 				)
@@
 			)
 		)
-		(property "Footprint" "Package_TO_SOT_THT:TO-92_Inline"
+		(property "Footprint" "Package_TO_SOT_THT:TO-92_Inline_Wide"
 			(at 81.28 64.135 0)
 			(hide yes)
@@
 			)
 		)
-		(property "Footprint" "Package_TO_SOT_THT:TO-92_Inline"
+		(property "Footprint" "Package_TO_SOT_THT:TO-92_Inline_Wide"
 			(at 199.39 155.575 0)
 			(hide yes)
@@
 			)
 		)
-		(property "Footprint" "Package_TO_SOT_THT:TO-92_Inline"
+		(property "Footprint" "Package_TO_SOT_THT:TO-92_Inline_Wide"
 			(at 147.32 36.195 0)
 			(hide yes)
@@
 			)
 		)
-		(property "Footprint" "Capacitor_THT:CP_Radial_D5.0mm_P2.50mm"
+		(property "Footprint" "Capacitor_THT:CP_Radial_D5.0mm_P2.00mm"
 			(at 35.56 118.11 0)
 			(hide yes)
@@
 			)
 		)
-		(property "Footprint" "Package_TO_SOT_THT:TO-92_Inline"
+		(property "Footprint" "Package_TO_SOT_THT:TO-92_Inline_Wide"
 			(at 171.45 36.195 0)
 			(hide yes)
@@
 			)
 		)
-		(property "Footprint" "Capacitor_THT:C_Rect_L7.0mm_W2.0mm_P5.00mm"
+		(property "Footprint" "Capacitor_THT:C_Rect_L7.0mm_W4.5mm_P5.00mm"
 			(at 140.97 153.67 0)
 			(hide yes)
@@
 			)
 		)
-		(property "Footprint" "Package_TO_SOT_THT:TO-92_Inline"
+		(property "Footprint" "Package_TO_SOT_THT:TO-92_Inline_Wide"
 			(at 54.61 130.175 0)
 			(hide yes)
