File: kicad/connections.kicad_sch (KiCad schematic)
At the start: 6 parts, among them J1 Conn_01x02_Pin, J2 Conn_01x02_Pin, J3 Conn_01x02_Pin, J4 Conn_01x02_Pin, J5 Conn_01x02_Pin, T1 Transformer_1P_1S

Commit message: Completed PCB
Parts:
- removed J1, J2, J3, J4, J5: Conn_01x02_Pin, TerminalBlock_4Ucon:TerminalBlock_4Ucon_1x02_P3.50mm_Horizontal, symbol Connector:Conn_01x02_Pin
- added J1, J10, J11, J12, J2, J3, J4, J5, J8, J9: (no value), ACRM:Spade_Connector, symbol ACRM:Spade_Connector
- T1: footprint Transformer_THT:Transformer_CHK_EI48-8VA_1xSec -> ACRM:Transformer_Myrra-44233-230V-18V-5VA-37x44
Connections:
- net AMP_LEFT: now also J3.1, J3.2
- net AMP_LEFT_GND: now also J10.1, J10.2, J4.1, J4.2
- net AMP_LEFT_OUT: now also J9.1, J9.2
- net AMP_RIGHT: now also J5.1, J5.2
- net AMP_RIGHT_GND: now also J12.1, J12.2, J8.1, J8.2
- net AMP_RIGHT_OUT: now also J11.1, J11.2
- net at T1.1 (AA): now also J1.1, J1.2
- net at T1.2 (AB): now also J2.1, J2.2
